Commit message: Fixed Keyboard node

File: urdf/kobuki.xacro (robot description, xacro)
@@ -43,4 +43,7 @@
     width="0.08"
     />
+    <gazebo reference="base">
+        <material>Gazebo/BlueGlow</material>
+    </gazebo>
     <xacro:wheel_joint name= "left_joint"
     origin_rpy = "$(eval -pi/2) 0 0"
@@ -58,4 +61,7 @@
     width = "0.021"
     />
+    <gazebo reference="left_wheel">
+        <material>Gazebo/FlatBlack</material>
+    </gazebo>
     <xacro:wheel_joint name= "right_joint"
     origin_rpy = "$(eval -pi/2) 0 0"
@@ -73,4 +79,7 @@
     width = "0.021"
     />
+    <gazebo reference="right_wheel">
+        <material>Gazebo/FlatBlack</material>
+    </gazebo>
     <xacro:fixed_joint name="back_joint"
     origin_xyz = "-0.115 0 -0.03"
@@ -85,4 +94,7 @@
     radius = "0.025"
     />
+    <gazebo reference="back_sphere">
+        <material>Gazebo/Grey</material>
+    </gazebo>
     <xacro:fixed_joint name="front_joint"
     origin_xyz = "0.115 0 -0.03"
@@ -97,4 +109,7 @@
     radius = "0.024"
     />
+    <gazebo reference="front_sphere">
+        <material>Gazebo/Grey</material>
+    </gazebo>
     <xacro:wheel_transmission name = "left_wheel_transmission"
     joint = "left_joint"
